Commit message: cam_stil_fail

File: src/ayn_simulation/ayn_description/urdf/depth_camera.xacro (robot description, xacro)
@@ -3,45 +3,25 @@
     <joint name="camera_joint" type="fixed">
         <parent link="base_link"/>
-        <child link="camera_frame"/>
-        <origin xyz="0 0 0.3" rpy="0 0 0"/>
+        <child link="camera_link"/>
+        <origin xyz="0.305 0 0.08" rpy="0 0 0"/>
     </joint>
-    <link name="camera_frame">
-        <!-- <visual>
+    <link name="camera_link">
+        <visual>
             <geometry>
-                <cylinder radius="0.05" length="0.06"/>
+                <box size="0.010 0.03 0.03"/>
             </geometry>
-            <material name="blue"/>
+            <material name="red"/>
         </visual>
-        <collision>
-            <geometry>
-                <cylinder radius="0.05" length="0.06"/>
-            </geometry>
-        </collision>
-        <xacro:inertial_cylinder mass="0.1" length="0.06" radius="0.05">
-            <origin xyz="0 0 0" rpy="0 0 0"/>
-        </xacro:inertial_cylinder> -->
     </link>
     <joint name="camera_optical_joint" type="fixed">
-        <parent link="camera_frame"/>
-        <child link="camera_optical_link"/>
-        <origin xyz="0.12 0 0" rpy="-1.5707 0 -1.5707"/>
+        <parent link="camera_link"/>
+        <child link="camera_link_optical"/>
+        <origin xyz="0 0 0" rpy="${-pi/2} 0 ${-pi/2}"/>
     </joint>
-    <link name="camera_optical_link">
-        <visual>
-            <geometry>
-                <box size="0.4 0.03 0.02"/>
-            </geometry>
-            <material name="blue"/>
-        </visual>
-        <collision>
-            <geometry>
-                <box size="0.4 0.03 0.02"/>
-            </geometry>
-        </collision>
-    </link>
-    <gazebo reference="camera_frame">
-        <material>Gazebo/Blue</material>
+    <link name="camera_link_optical"></link>
+    <gazebo reference="camera_link">
+        <material>Gazebo/Red</material>
         <sensor name="camera" type="depth">
-            <pose>0.064 -0.065 0.094  0 0 0 </pose>
+            <pose> 0 0 0 0 0 0 </pose>
             <visualize>true</visualize>
             <update_rate>10</update_rate>
@@ -58,13 +38,9 @@
                 </clip>
             </camera>
-            <!-- <plugin name="camera_controller" filename="libgazebo_ros_camera.so">
-                <frame_name>camera_optical_link</frame_name>
-            </plugin> -->
             <plugin name="camera_controller" filename="libgazebo_ros_camera.so">
-            <cameraName>camera</cameraName>
-            <frameName>camera_optical_link</frameName>
-            <imageTopicName>image_raw</imageTopicName>
-            <cameraInfoTopicName>camera_info</cameraInfoTopicName>
-        </plugin>
+                <frame_name>camera_link_optical</frame_name>
+                <min_depth>0.1</min_depth>
+                <max_depth>100.0</max_depth>
+            </plugin>
         </sensor>
     </gazebo>

File: src/ayn_simulation/ayn_description/urdf/robot.urdf.xacro (robot description, xacro)
@@ -9,5 +9,3 @@
     <xacro:include filename="camera.xacro" /> -->
     <xacro:include filename="depth_camera.xacro" />
-    <xacro:include filename="gps.xacro" />
-    <xacro:include filename="imu.xacro" />
 </robot>

Commit message: Depth_camera::OK

File: src/ayn_simulation/ayn_description/urdf/depth_camera.xacro (robot description, xacro)
@@ -1,47 +1,70 @@
 <?xml version="1.0"?>
-<robot xmlns:xacro="http://www.ros.org/wiki/xacro" >
-    <joint name="camera_joint" type="fixed">
-        <parent link="base_link"/>
-        <child link="camera_link"/>
-        <origin xyz="0.305 0 0.08" rpy="0 0 0"/>
-    </joint>
-    <link name="camera_link">
-        <visual>
-            <geometry>
-                <box size="0.010 0.03 0.03"/>
-            </geometry>
-            <material name="red"/>
-        </visual>
-    </link>
-    <joint name="camera_optical_joint" type="fixed">
-        <parent link="camera_link"/>
-        <child link="camera_link_optical"/>
-        <origin xyz="0 0 0" rpy="${-pi/2} 0 ${-pi/2}"/>
-    </joint>
-    <link name="camera_link_optical"></link>
-    <gazebo reference="camera_link">
-        <material>Gazebo/Red</material>
-        <sensor name="camera" type="depth">
-            <pose> 0 0 0 0 0 0 </pose>
-            <visualize>true</visualize>
-            <update_rate>10</update_rate>
-            <camera>
-                <horizontal_fov>1.089</horizontal_fov>
-                <image>
-                    <format>B8G8R8</format>
-                    <width>640</width>
-                    <height>480</height>
-                </image>
-                <clip>
-                    <near>0.05</near>
-                    <far>8.0</far>
-                </clip>
-            </camera>
-            <plugin name="camera_controller" filename="libgazebo_ros_camera.so">
-                <frame_name>camera_link_optical</frame_name>
-                <min_depth>0.1</min_depth>
-                <max_depth>100.0</max_depth>
-            </plugin>
-        </sensor>
-    </gazebo>
+<robot xmlns:xacro="http://www.ros.org/wiki/xacro">
+  <!-- Mount camera to base -->
+  <joint name="camera_joint" type="fixed">
+    <parent link="base_link"/>
+    <child link="camera_link"/>
+    <origin xyz="0.305 0 0.08" rpy="0 0 0"/>
+  </joint>
+  <link name="camera_link">
+    <visual>
+      <geometry>
+        <box size="0.010 0.03 0.03"/>
+      </geometry>
+      <material name="red"/>
+    </visual>
+    <collision>
+      <geometry>
+        <box size="0.010 0.03 0.03"/>
+      </geometry>
+    </collision>
+    <inertial>
+      <mass value="0.1"/>
+      <origin xyz="0 0 0" rpy="0 0 0"/>
+      <inertia ixx="1e-5" ixy="0" ixz="0" iyy="1e-5" iyz="0" izz="1e-5"/>
+    </inertial>
+  </link>
+  <!-- Optical frame (for proper TF alignment) -->
+  <joint name="camera_optical_joint" type="fixed">
+    <parent link="camera_link"/>
+    <child link="camera_link_optical"/>
+    <origin xyz="0 0 0" rpy="${-pi/2} 0 ${-pi/2}"/>
+  </joint>
+  <link name="camera_link_optical">
+    <inertial>
+      <mass value="0.001"/>
+      <origin xyz="0 0 0" rpy="0 0 0"/>
+      <inertia ixx="1e-6" ixy="0" ixz="0" iyy="1e-6" iyz="0" izz="1e-6"/>
+    </inertial>
+  </link>
+  <!-- Attach the Gazebo depth sensor to the optical frame -->
+  <gazebo reference="camera_link_optical">
+    <sensor name="depth_camera" type="depth">
+      <pose>0 0 0 0 0 0</pose>
+      <visualize>true</visualize>
+      <update_rate>30</update_rate>
+      <camera>
+        <horizontal_fov>1.089</horizontal_fov>
+        <image>
+          <format>R8G8B8</format>
+          <width>640</width>
+          <height>480</height>
+        </image>
+        <clip>
+          <near>0.05</near>
+          <far>8.0</far>
+        </clip>
+      </camera>
+      <plugin name="gazebo_ros_depth_camera" filename="libgazebo_ros_depth_camera.so">
+        <ros>
+          <namespace>/camera</namespace>
+        </ros>
+        <frame_name>camera_link_optical</frame_name>
+        <image_topic_name>image_raw</image_topic_name>
+        <depth_image_topic_name>depth/image_raw</depth_image_topic_name>
+        <depth_camera_info_topic_name>depth/camera_info</depth_camera_info_topic_name>
+        <point_cloud_topic_name>depth/points</point_cloud_topic_name>
+      </plugin>
+    </sensor>
+  </gazebo>
 </robot>
